File: v01/comm_circuit.sch (KiCad schematic (older format))
At the start: 17 parts

Commit message: ERC.
Parts:
- removed C?: 0.1uF, ~, symbol C
- gave numbers to parts that had none: 16
Connections:
- net +5V: no longer R19.2, R21.2, R22.2, R24.2
- net +3.3V renamed 3.3V
- net 3V3_USB: no longer names the net of U3.17 (3V3OUT)
- new net VBAT: R19.2, R21.2, R22.2, R24.2
- no-connect marks 13 -> 14
Other:
- note added: "Had to make Vbus of the USB connector an input pin \nbecause the power flag connected to +5V is considered \nan output pin."
