File: v02_R/volt_reg_batt_chg.sch (KiCad schematic (older format))
At the start: 14 parts, among them P1 CONN_1, P2 CONN_1, Q3 PNP, SW1 SW_PUSH_SMALL, U3 TPS73601DBVR

Commit message: Update -- order submitted to OSHPark
Parts:
- R28: value 0.8 -> 2
Other:
- note added: "CSR8675 datasheet suggests a 400 milliohm resistor \nto get a charge current of 500 mA. They say that a \nLi-Ion battery should be charged < 1 C, hence a \n150 mAh battery should be given no more than 150 \nmA constant charge current. I'm raising the resistance \nto 5*400 milliohm = 2 ohm. I'm thinking this should\nlimit the constant charge current to about 100 mA."
Changed lines of the file:
@@
 Sheet 4 4
 Title ""
-Date "28 jan 2015"
+Date "26 feb 2015"
 Rev ""
 Comp ""
@@
 P 2600 5150
 F 0 "R28" V 2680 5150 40  0000 C CNN
-F 1 "0.8" V 2607 5151 40  0000 C CNN
+F 1 "2" V 2607 5151 40  0000 C CNN
 F 2 "~" V 2530 5150 30  0000 C CNN
 F 3 "~" H 2600 5150 30  0000 C CNN
@@
 	5500 2250 5500 1850
 Connection ~ 5500 1850
+Text Notes 3150 5100 0    60   ~ 0
+CSR8675 datasheet suggests a 400 milliohm resistor \nto get a charge current of 500 mA. They say that a \nLi-Ion battery should be charged < 1 C, hence a \n150 mAh battery should be given no more than 150 \nmA constant charge current. I'm raising the resistance \nto 5*400 milliohm = 2 ohm. I'm thinking this should\nlimit the constant charge current to about 100 mA.
 $EndSCHEMATC
