File: v01_R/_autosave-CWIEM_PCB_v01_R.kicad_pcb (KiCad board)
At the start: 2 copper layers, 0 parts

Commit message: Submitting the latest stuff.
Parts:
- added C1: 10uF, SM0805, F.Cu at (72.6, 85.9)
- added C10: 47pF, SM0402_c, F.Cu at (64.5, 71.1)
- added C11: 0.1uF, SM0402_c, F.Cu at (60.7, 72.9)
- added C12: 1.0uF, SM0402_c, F.Cu at (70.6, 73.2)
- added C13: 180pF, SM0402_c, F.Cu at (64.3, 73.7)
- added C14: 0.1uF, SM0402_c, F.Cu at (60.7, 74.2)
- added C15: 47pF, SM0402_c, F.Cu at (68.6, 74.4)
- added C16: 1.5uF, SM0402_c, F.Cu at (70.1, 76.2)
- added C17: 3.3uF, SM0402_c, F.Cu at (75.6, 78.9)
- added C18: 10uF, SM0805, F.Cu at (91.5, 79.2)
- added C19: 0.1uF, SM0402_c, F.Cu at (91.5, 73.4)
- added C2: 1uF, SM0402_c, F.Cu at (82.8, 85.3)
- added C20: 4.7uF, SM0402_c, F.Cu at (70.1, 83.1)
- added C3: 10uF, SM0805, F.Cu at (84.8, 86.9)
- added C6: 1.0uF, SM0402_c, F.Cu at (66.5, 59.2)
- added C9: 1.0uF, SM0402_c, F.Cu at (69.1, 63.8)
- added D2: LED, LED-0603, F.Cu at (86.8, 66.8)
- added D3: LED, LED-0603, F.Cu at (86.9, 70.1)
- added J1: USB, conn_usb_B_micro_smd, F.Cu at (98.0, 74.7)
- added P1: CONN_1, BA Driver Pad, F.Cu at (78.2, 82.3)
- added P12: CONN_1, ci_pad, F.Cu at (78.7, 76.3)
- added P2: CONN_1, BA Driver Pad, B.Cu at (79.0, 59.4)
- added P7: CONN_1, wbfk_pad, F.Cu at (74.7, 73.7)
- added P8: CONN_1, wbfk_pad, F.Cu at (76.1, 73.7)
- added P9: CONN_1, ci_pad, F.Cu at (75.2, 76.3)
- added Q3: PNP, SOT23EBC, F.Cu at (68.2, 88.0)
- added R1: 52.3k, SM0402_r, F.Cu at (81.3, 85.3)
- added R12: 30.1k, SM0402_r, F.Cu at (62.2, 71.1)
- added R13: 15k, SM0402_r, F.Cu at (62.7, 72.9)
- added R14: 43k, SM0402_r, F.Cu at (65.8, 72.9)
- added R15: 15k, SM0402_r, F.Cu at (62.7, 74.2)
- added R16: 43k, SM0402_r, F.Cu at (65.8, 74.2)
- added R17: 30.1k, SM0402_r, F.Cu at (70.6, 74.4)
- added R18: 20, SM0805, F.Cu at (68.3, 77.0)
- added R2: 30.1k, SM0402_r, F.Cu at (81.3, 87.4)
- added R27: 10k, SM0402_r, F.Cu at (62.7, 85.6)
- added R28: 0.8, SM0805, F.Cu at (67.3, 85.1)
- added R29: 0.15, SM0805, F.Cu at (67.3, 83.1)
- added R3: 240, SM0402_r, F.Cu at (86.8, 63.8)
- added R4: 240, SM0402_r, F.Cu at (86.4, 72.6)
- added SW1: SW_PUSH_SMALL, SW_PUSH_SMD, B.Cu at (77.7, 92.2)
- added U1: BC127, BC127, F.Cu at (73.4, 54.4)
- added U2: TI_TPA6138A2, TSSOP14, F.Cu at (65.8, 63.8)
- added U3: TPS73601DBVR, SOT23-5, F.Cu at (78.2, 85.9)
Routing:
- net GND: track 0.00 -> 82.8 mm, vias 0 -> 9
- net 3.3V: track 0.00 -> 81.4 mm, vias 0 -> 3
- net 5V_USB: track 0.00 -> 52.8 mm
- net VBAT: track 0.00 -> 47.5 mm
- net VREGEN: track 0.00 -> 46.5 mm, vias 0 -> 1
- net CHG_EXT: track 0.00 -> 37.9 mm
- net VBAT_SENSE: track 0.00 -> 30.6 mm, vias 0 -> 2
- net AIO_1: track 0.00 -> 29.4 mm, vias 0 -> 2
- net SPKR_RN: track 0.00 -> 22.2 mm, vias 0 -> 2
- net SPKR_RP: track 0.00 -> 16.8 mm, vias 0 -> 2
- net N-0000062: track 0.00 -> 13.9 mm
- net N-0000052: track 0.00 -> 12.4 mm, vias 0 -> 2
- net N-0000061: track 0.00 -> 11.4 mm
- net N-0000051: track 0.00 -> 11.3 mm
- net N-0000050: track 0.00 -> 9.08 mm
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- added copper zone on B.Cu, net GND
- added copper zone on F.Cu, net GND
Other:
- board outline added: 45.7 x 45.7 mm
- rule pad_to_mask_clearance: 0 -> 0.0508
- board text added: "CWIEM R v01"
